File: Starbie.kicad_sch (KiCad schematic)
At the start: 7 parts, among them J1 Conn_01x04_Pin, J2 Conn_01x08_Pin, SW1 SW_Push, SW2 SW_Push, U1 XIAO-ESP32-C3-SMD, U2 DHT11

Commit message: Added pcb and sch files to github
Parts:
- added C1, C2: 0.1uF, Capacitor_SMD:C_0402_1005Metric, symbol Device:C
- added C3: 10uF, Capacitor_SMD:C_0805_2012Metric, symbol Device:C
- added LS1: Speaker, Package_DFN_QFN:TQFN-16-1EP_3x3mm_P0.5mm_EP1.23x1.23mm, symbol Device:Speaker
- added MK1: ICS-43434, Sensor_Audio:InvenSense_ICS-43434-6_3.5x2.65mm, symbol Sensor_Audio:ICS-43434
- added U3: MAX98357A, Package_DFN_QFN:TQFN-16-1EP_3x3mm_P0.5mm_EP1.23x1.23mm, symbol Audio:MAX98357A
Connections:
- net +3.3V: now also C1.1, C2.1, C3.1, MK1.5 (VDD), U3.7 (VDD), U3.8 (VDD)
- net +5V: now also U3.4 (~{SD_MODE})
- net DHT11 DATA: now also U1.3 (D2); no longer U1.2 (D1)
- net GND: now also C1.2, C2.2, C3.2, MK1.2 (LR), MK1.3 (GND), U3.11 (GND), U3.15 (GND), U3.17 (PAD), U3.3 (GND)
- net GP102: now also U1.4 (D3); no longer U1.3 (D2)
- net GP103: now also U1.5 (D4); no longer U1.4 (D3)
- net SCL: now also U1.6 (D5); no longer U1.5 (D4)
- net SDA: now also U1.7 (D6); no longer U1.6 (D5)
- net WS: now reaches U1.11 (D10)
- net WS: now also MK1.1 (WS), U3.14 (LRCLK)
- net SD: now reaches U1.8 (D7)
- net SD: now also MK1.6 (SD)
- net DIN: now reaches U1.9 (D8)
- net DIN: now also U3.1 (DIN)
- new net: LS1.2, U3.10 (OUTN)
- new net: LS1.1, U3.9 (OUTP)
- new net SCK: MK1.4 (SCK), U1.2 (D1), U3.16 (BCLK)
- no-connect marks 18 -> 14
